File: RAM tester/kicad/ram_tester/ram_tester.kicad_pcb (KiCad board)
At the start: 2 copper layers, 253 x 124.2 mm, 22 parts, among them J1 Conn_01x04_Male, SW1 SW_Push, U1 fubarino_sd

Commit message: Add files via upload
Parts:
- moved R9 68.1 mm to (98.2, 52.2)
- moved SW1 65.8 mm to (98.2, 30.6), turned to 90 degrees
- moved DS1 28.3 mm to (133.9, -10.7)
- moved J1 25.6 mm to (116.3, 23.3)
- moved R1 25.4 mm to (90.8, 42.0)
- moved R2 25.4 mm to (85.0, 42.3)
- moved R5 25.4 mm to (66.8, 42.3)
- moved R6 25.4 mm to (60.9, 42.3)
- moved D1 25.4 mm to (91.0, 35.1)
- moved D2 25.4 mm to (85.0, 35.1)
- moved D3 25.4 mm to (79.0, 35.1)
- moved D4 25.4 mm to (72.9, 35.1)
- moved D5 25.4 mm to (66.8, 35.1)
- moved D6 25.4 mm to (60.8, 35.1)
- moved D7 25.4 mm to (54.8, 35.1)
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Routing:
- net +3.3V: track 145.9 -> 233.5 mm
- net Net-(U1A-36/A8): track 146.9 -> 232.4 mm
- net Net-(J1-Pin_2): track 136.8 -> 168.0 mm
- net GND: track 350.0 -> 379.8 mm
- net Net-(J1-Pin_1): track 155.0 -> 182.5 mm
- net Net-(D1-A): track 113.5 -> 138.8 mm
- net Net-(D8-A): track 131.7 -> 157.1 mm
- net Net-(D7-A): track 129.7 -> 155.0 mm
- net Net-(D6-A): track 126.7 -> 152.1 mm
- net Net-(D4-A): track 122.8 -> 148.2 mm
- net Net-(D3-A): track 121.1 -> 146.5 mm
- net Net-(D2-A): track 117.4 -> 142.7 mm
- net Net-(D5-A): track 123.9 -> 149.2 mm
- net +5V: track 369.2 -> 391.8 mm
Other:
- board size 253 x 124.2 mm -> 253 x 150.6 mm
